File: xmas-badge.sch (KiCad schematic (older format))
At the start: 13 parts, among them U1 BAT_HLD_2032, U2 LP, U3 LP, U4 LP, U5 LP

Commit message: first small version
Parts:
- D1: symbol !Goody:LED -> xmas-badge-rescue:LED-!Goody
- R1, R2, R3, R4, R5, R6: symbol !Goody:R -> xmas-badge-rescue:R-!Goody
- S1: symbol !Goody:Micro_Schalter -> xmas-badge-rescue:Micro_Schalter-!Goody
- U1: symbol !Goody:BAT_HLD_2032 -> xmas-badge-rescue:BAT_HLD_2032-!Goody
- U2, U3, U4, U5: symbol !Goody:LP -> xmas-badge-rescue:LP-!Goody
Changed lines of the file:
@@
 encoding utf-8
 Sheet 1 1
-Title ""
-Date ""
-Rev ""
-Comp ""
-Comment1 ""
+Title "XMas Badge"
+Date "2021-10-23"
+Rev "1.0.0"
+Comp "FabLab Oberland e.V."
+Comment1 "Karlheinz Frank & Alexander Kutschera"
 Comment2 ""
 Comment3 ""
@@
 $EndDescr
 $Comp
-L !Goody:BAT_HLD_2032 U1
+L xmas-badge-rescue:BAT_HLD_2032-!Goody U1
 U 1 1 6152D3A3
 P 2500 2600
@@
 $EndComp
 $Comp
-L !Goody:Micro_Schalter S1
+L xmas-badge-rescue:Micro_Schalter-!Goody S1
 U 1 1 6152DBDE
 P 3250 1750
@@
 $EndComp
 $Comp
-L !Goody:R R4
+L xmas-badge-rescue:R-!Goody R4
 U 1 1 6152DEF1
 P 5600 1750
@@
 $EndComp
 $Comp
-L !Goody:R R5
+L xmas-badge-rescue:R-!Goody R5
 U 1 1 6152EAC1
 P 5600 2000
@@
 $EndComp
 $Comp
-L !Goody:R R6
+L xmas-badge-rescue:R-!Goody R6
 U 1 1 6152EC15
 P 6600 1850
@@
 $EndComp
 $Comp
-L !Goody:R R1
+L xmas-badge-rescue:R-!Goody R1
 U 1 1 6152ED79
 P 3800 3600
@@
 $EndComp
 $Comp
-L !Goody:R R3
+L xmas-badge-rescue:R-!Goody R3
 U 1 1 6152EEED
 P 4700 3600
@@
 $EndComp
 $Comp
-L !Goody:R R2
+L xmas-badge-rescue:R-!Goody R2
 U 1 1 6152F071
 P 4300 3950
@@
 $EndComp
 $Comp
-L !Goody:LED D1
+L xmas-badge-rescue:LED-!Goody D1
 U 1 1 6152F28A
 P 8000 2550
@@
 $EndComp
 $Comp
-L !Goody:LP U4
+L xmas-badge-rescue:LP-!Goody U4
 U 1 1 6152F9D0
 P 5450 1450
@@
 $EndComp
 $Comp
-L !Goody:LP U5
+L xmas-badge-rescue:LP-!Goody U5
 U 1 1 6152FD38
 P 5750 1450
@@
 $EndComp
 $Comp
-L !Goody:LP U2
+L xmas-badge-rescue:LP-!Goody U2
 U 1 1 615305BB
 P 4550 3350
@@
 $EndComp
 $Comp
-L !Goody:LP U3
+L xmas-badge-rescue:LP-!Goody U3
 U 1 1 615305C1
 P 4850 3350

Commit message: saved
Parts:
- S1: footprint KHF_LIB:Micro_SchalterKHF -> libraries:Micro_SchalterKHF
- U1: footprint Battery:BatteryHolder_Keystone_106_1x20mm -> libraries:BAT-HLD-012-SMT
- U2, U3, U4, U5: footprint KHF_LIB:LP -> libraries:LP
Changed lines of the file:
@@
 F 0 "U1" H 2387 2665 50  0000 C CNN
 F 1 "BAT_HLD_2032" H 2387 2574 50  0000 C CNN
-F 2 "Battery:BatteryHolder_Keystone_106_1x20mm" H 2387 2483 50  0000 C CNN
+F 2 "libraries:BAT-HLD-012-SMT" H 2387 2483 50  0000 C CNN
 F 3 "" H 2050 2200 50  0001 C CNN
 	1    2500 2600
@@
 F 0 "S1" H 3458 1609 50  0000 L CNN
 F 1 "Micro_Schalter" H 3250 1950 50  0001 C CNN
-F 2 "KHF_LIB:Micro_SchalterKHF" H 3458 1518 50  0000 L CNN
+F 2 "libraries:Micro_SchalterKHF" H 3458 1518 50  0000 L CNN
 F 3 "" H 3250 1750 50  0001 C CNN
 	1    3250 1750
@@
 F 0 "U4" V 5225 1337 50  0000 C CNN
 F 1 "LP" V 5316 1337 50  0000 C CNN
-F 2 "KHF_LIB:LP" H 5300 1800 50  0001 C CNN
+F 2 "libraries:LP" H 5300 1800 50  0001 C CNN
 F 3 "" H 5300 1800 50  0001 C CNN
 	1    5450 1450
@@
 F 0 "U5" H 5662 1291 50  0000 R CNN
 F 1 "LP" H 5662 1382 50  0000 R CNN
-F 2 "KHF_LIB:LP" H 5600 1800 50  0001 C CNN
+F 2 "libraries:LP" H 5600 1800 50  0001 C CNN
 F 3 "" H 5600 1800 50  0001 C CNN
 	1    5750 1450
@@
 F 0 "U2" V 4325 3237 50  0000 C CNN
 F 1 "LP" V 4416 3237 50  0000 C CNN
-F 2 "KHF_LIB:LP" H 4400 3700 50  0001 C CNN
+F 2 "libraries:LP" H 4400 3700 50  0001 C CNN
 F 3 "" H 4400 3700 50  0001 C CNN
 	1    4550 3350
@@
 F 0 "U3" H 4762 3191 50  0000 R CNN
 F 1 "LP" H 4762 3282 50  0000 R CNN
-F 2 "KHF_LIB:LP" H 4700 3700 50  0001 C CNN
+F 2 "libraries:LP" H 4700 3700 50  0001 C CNN
 F 3 "" H 4700 3700 50  0001 C CNN
 	1    4850 3350
